File: payload/pcb/IREC_HeatTransfer_Payload/IREC_HeatTransfer_Payload.kicad_sch (KiCad schematic)
At the start: 47 parts, among them J1 Screw_Terminal_01x06, J2 XT60PW-M, J3 Screw_Terminal_01x06, J4 Conn_01x04, J5 GPIO, J6 SPI, J7 I2C, U1 MAX31855KASA, U2 MAX31855KASA, U3 MAX31855KASA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

Commit message: upd
Parts:
- added JP2: Jumper_2_Open, CustomFootprintLib:SolderJumper, symbol Jumper:Jumper_2_Open
- J4: value Conn_01x04 -> POWER
Connections:
- net GND: now also JP2.2 (B); no longer H1.1, H2.1, H3.1, H4.1
- new net: H4.1, JP2.1 (A)
- no-connect marks 1 -> 4
Other:
- note added: "04/23/2024"
- note added: "1.0"
- note added: "Designed By: Luca Beretta"
- note added: "Extra Pins"
- note added: "Heat Transfer Board for Perception"
- note added: "Mounting Holes"
- note added: "VIN: 3.6V-5.5V Current Draw: 100mA"
- note removed: "VIN: 3.6V-5.5V"
- moved on the sheet: C1, C10, C13, C2, C3, C5, C6, C7, D1, D2, H1, H2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

Commit message: upd
Connections:
- no-connect marks 4 -> 6
Other:
- note added: "2.54mm Pin Headers"
Changed lines of the file:
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@@
+	)
+	(no_connect
+		(at 224.79 53.34)
 	)
 	(no_connect
 		(at 153.67 176.53)
+	)
+	(no_connect
+		(at 224.79 50.8)
 	)
 	(no_connect
@@
 	(rectangle
 		(start 15.24 170.18)
-		(end 53.34 231.14)
+		(end 53.34 233.68)
 		(stroke
 			(width 0)
@@
 		)
 	)
+	(text "2.54mm Pin Headers"
+		(exclude_from_sim no)
+		(at 42.418 232.156 0)
+		(effects
+			(font
+				(size 1.27 1.27)
+			)
+		)
+	)

Commit message: added pitot
Parts:
- added C14: 470pF, symbol Device:C
- added C15: 1.0uF, symbol Device:C
- added C16: 0.01uF, symbol Device:C
- added U8: MPXV7002DP, SnapEDA Library:XDCR_MPXV7002DP, symbol CustomComponents:MPXV7002DP
Connections:
- net +5V: now also U4.2 (EN), C15.1, C16.1, U8.2 (VS)
- net GND: now also C14.2, C15.2, C16.2, U8.3 (GND); no longer U4.4 (COMP), U4.8 (GND)
- net V_BUCK: no longer U4.1 (VIN), U4.2 (EN)
- net at C8.1: no longer U4.6 (BST)
- net at C8.2, L1.1: no longer U4.9 (SW)
- net at C9.2, R4.2, R5.1: now also U4.4 (COMP); no longer U4.3 (FB)
- net PITOT: now reaches U7.16 (A2)
- net PITOT: now also C14.1, U8.4 (VOUT)
Other:
- note added: "Pitot Tube"
- moved on the sheet: U4

Commit message: upd
Connections:
- net +5V: no longer U4.2 (EN)
- net GND: now also U4.4 (COMP), U4.8 (GND)
- net I2C_SCL: now also U7.19 (A5)
- net I2C_SDA: now also U7.18 (A4)
- net LED_GREEN: now also U7.41 (A17)
- net T1_CS: now also U7.20 (A6)
- net T2_CS: now also U7.21 (A7)
- net T3_CS: now also U7.22 (A8)
- net V_BUCK: now also U4.1 (VIN), U4.2 (EN)
- net at C8.1: now also U4.6 (BST)
- net at C8.2, L1.1: now also U4.9 (SW)
- net at U4.3 (FB): now also C9.2, R4.2, R5.1
- net MOSI: now reaches U7.11 (MOSI)
- net LED_RED: no longer names the net of U7.2 (OUT2)
- net TEMP_SENSE renamed DS18_TEMP
- net VBAT_CR2032 renamed VBAT_COIN
Other:
- moved on the sheet: U4
Changed lines of the file:
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@@
 	(paper "A3")
 	(junction
-		(at 125.73 50.8)
-		(diameter 0)
-		(color 0 0 0 0)
-	)
-	(junction
 		(at 129.54 50.8)
 		(diameter 0)
@@
 	)
 	(junction
+		(at 95.25 35.56)
+		(diameter 0)
+		(color 0 0 0 0)
+	)
+	(junction
 		(at 93.98 58.42)
 		(diameter 0)
@@
 	(junction
 		(at 267.97 134.62)
-		(diameter 0)
-		(color 0 0 0 0)
-	)
-	(junction
-		(at 125.73 43.18)
 		(diameter 0)
 		(color 0 0 0 0)
@@
 	(wire
 		(pts
-			(xy 125.73 50.8) (xy 129.54 50.8)
-		)
-		(stroke
-			(width 0)
-			(type default)
-		)
-	)
-	(wire
-		(pts
 			(xy 39.37 110.49) (xy 41.91 110.49)
 		)
@@
 	(wire
 		(pts
-			(xy 115.57 50.8) (xy 125.73 50.8)
+			(xy 115.57 50.8) (xy 129.54 50.8)
 		)
 		(stroke
@@
 	(rectangle
 		(start 15.24 125.73)
-		(end 58.42 165.1)
+		(end 60.96 165.1)
 		(stroke
 			(width 0)
@@
 		)
 	)
-	(label "T2_CS"
-		(at 334.01 78.74 0)
-		(fields_autoplaced yes)
-		(effects
-			(font
-				(size 1.27 1.27)
-			)
-			(justify left bottom)
-		)
-	)
-	(label "T1_CS"
-		(at 334.01 43.18 0)
-		(fields_autoplaced yes)
-		(effects
-			(font
-				(size 1.27 1.27)
-			)
-			(justify left bottom)
-		)
-	)
-	(label "T3_CS"
-		(at 334.01 114.3 0)
-		(fields_autoplaced yes)
-		(effects
-			(font
-				(size 1.27 1.27)
-			)
-			(justify left bottom)
-		)
-	)
-	(label "SCK"
-		(at 334.01 35.56 0)
-		(fields_autoplaced yes)
-		(effects
-			(font
-				(size 1.27 1.27)
-			)
-			(justify left bottom)
-		)
-	)
 	(global_label "V_BUCK"
 		(shape output)
@@
 		)
 	)
-	(hierarchical_label "VBAT_CR2032"
+	(hierarchical_label "VBAT_COIN"
 		(shape output)
 		(at 193.04 67.31 0)
@@
 	(hierarchical_label "SCK"
 		(shape input)
+		(at 334.01 35.56 0)
+		(fields_autoplaced yes)
+		(effects
+			(font
+				(size 1.27 1.27)
+			)
+			(justify left)
+		)
+	)
+	(hierarchical_label "SCK"
+		(shape input)
 		(at 334.01 106.68 0)
 		(fields_autoplaced yes)
@@
 		)
 	)
+	(hierarchical_label "T1_CS"
+		(shape output)
+		(at 334.01 43.18 0)
+		(fields_autoplaced yes)
+		(effects
+			(font
+				(size 1.27 1.27)
+			)
+			(justify left)
+		)
+	)
 	(hierarchical_label "T1"
 		(shape output)
@@
 		)
 	)
+	(hierarchical_label "I2C_SCL"
+		(shape input)
+		(at 224.79 111.76 180)
+		(fields_autoplaced yes)
+		(effects
+			(font
+				(size 1.27 1.27)
+			)
+			(justify right)
+		)
+	)
 	(hierarchical_label "MISO"
 		(shape output)
@@
 		)
 	)
-	(hierarchical_label "TEMP_SENSE"
+	(hierarchical_label "DS18_TEMP"
 		(shape input)
 		(at 224.79 99.06 180)
@@
 			)
 			(justify right)
+		)
+	)
+	(hierarchical_label "MOSI"
+		(shape output)
+		(at 265.43 96.52 0)
+		(fields_autoplaced yes)
+		(effects
+			(font
+				(size 1.27 1.27)
+			)
+			(justify left)
 		)
 	)
@@
 	)
 	(hierarchical_label "PITOT"
-		(shape output)
+		(shape input)
 		(at 224.79 104.14 180)
+		(fields_autoplaced yes)
+		(effects
+			(font
+				(size 1.27 1.27)
+			)
+			(justify right)
+		)
+	)
+	(hierarchical_label "I2C_SDA"
+		(shape input)
+		(at 224.79 109.22 180)
 		(fields_autoplaced yes)
 		(effects
@@
 		)
 	)
-	(hierarchical_label "VBAT_CR2032"
+	(hierarchical_label "VBAT_COIN"
 		(shape input)
 		(at 265.43 43.18 0)
@@
 		)
 	)
-	(hierarchical_label "TEMP_SENSE"
+	(hierarchical_label "T1_CS"
+		(shape input)
+		(at 224.79 114.3 180)
+		(fields_autoplaced yes)
+		(effects
+			(font
+				(size 1.27 1.27)
+			)
+			(justify right)
+		)
+	)
+	(hierarchical_label "DS18_TEMP"
 		(shape output)
 		(at 44.45 149.86 0)
@@
 		)
 	)
+	(hierarchical_label "T3_CS"
+		(shape output)
+		(at 334.01 114.3 0)
+		(fields_autoplaced yes)
+		(effects
+			(font
+				(size 1.27 1.27)
+			)
+			(justify left)
+		)
+	)
 	(hierarchical_label "VBAT_SENSE"
 		(shape output)
@@
 		)
 	)
+	(hierarchical_label "T3_CS"
+		(shape input)
+		(at 224.79 119.38 180)
+		(fields_autoplaced yes)
+		(effects
+			(font
+				(size 1.27 1.27)
+			)
+			(justify right)
+		)
+	)
+	(hierarchical_label "T2_CS"
+		(shape output)
+		(at 334.01 78.74 0)
+		(fields_autoplaced yes)
+		(effects
+			(font
+				(size 1.27 1.27)
+			)
+			(justify left)
+		)
+	)
 	(hierarchical_label "T3"
 		(shape output)
@@
 		)
 	)
+	(hierarchical_label "T2_CS"
+		(shape input)
+		(at 224.79 116.84 180)
+		(fields_autoplaced yes)
+		(effects
+			(font
+				(size 1.27 1.27)
+			)
+			(justify right)
+		)
+	)
 	(hierarchical_label "GPIO"
 		(shape bidirectional)
@@
 		)
 	)
-	(hierarchical_label "LED_RED"
-		(shape output)
-		(at 265.43 71.12 0)
-		(fields_autoplaced yes)
-		(effects
-			(font
-				(size 1.27 1.27)
-			)
-			(justify left)
-		)
-	)
 	(hierarchical_label "T2"
 		(shape input)
 		(at 133.35 135.89 0)
+		(fields_autoplaced yes)
+		(effects
+			(font
+				(size 1.27 1.27)
+			)
+			(justify left)
+		)
+	)
+	(hierarchical_label "LED_GREEN"
+		(shape output)
+		(at 265.43 104.14 0)
 		(fields_autoplaced yes)
 		(effects
@@
 		(lib_id "CustomComponents:AP63357_(SparkFun_Buck_Regulator_5V)")
 		(at 110.49 53.34 0)
-		(mirror y)
 		(unit 1)
 		(exclude_from_sim no)
@@
 		(dnp no)
 		(property "Reference" "U4"
-			(at 115.57 25.146 0)
+			(at 105.41 25.146 0)
 			(effects
 				(font
@@
 		)
 		(property "Value" "AP63357"
-			(at 115.57 28.448 0)
-			(effects
-				(font
+			(at 105.41 28.448 0)
+			(effects
+				(font

Commit message: updates
Parts:
- added J9: Serial, Connector_PinSocket_2.54mm:PinSocket_1x02_P2.54mm_Vertical, symbol Connector_Generic:Conn_01x02
- J2: footprint CustomFootprintLib:AMASS_XT60PW-M -> Connector_AMASS:AMASS_XT60-M_1x02_P7.20mm_Vertical
Connections:
- net MOSI is gone; now on net SPI_MOSI: U7.11 (MOSI)
- net +3V3: now also J4.3 (Pin_3); no longer J4.2 (Pin_2)
- net +5V: now also J4.2 (Pin_2); no longer J4.1 (Pin_1)
- net I2C_SCL: now also J7.1 (Pin_1); no longer J7.2 (Pin_2)
- net I2C_SDA: now also J7.2 (Pin_2); no longer J7.1 (Pin_1)
- net LED_GREEN: now also U7.23 (A9); no longer U7.3 (LRCLK2), U7.41 (A17)
- net MISO: no longer U7.12 (MISO)
- net SPI_MISO: now also J6.2 (Pin_2), U7.12 (MISO); no longer J6.3 (Pin_3)
- net SPI_MOSI: now also J6.3 (Pin_3); no longer J6.2 (Pin_2)
- net VCC: now also J4.1 (Pin_1); no longer J4.3 (Pin_3)
- net RX: now reaches U7.0 (RX1)
- net RX: now also J9.1 (Pin_1)
- net TX: now reaches U7.1 (TX1)
- net TX: now also J9.2 (Pin_2)
- net GPIO2: now reaches U7.2 (OUT2)
- net GPIO2: now also J5.1 (Pin_1)
- net GPIO4: now reaches U7.4 (BCLK2)
- net GPIO4: now also J5.3 (Pin_3)
- net GPIO5: now reaches U7.5 (IN2)
- net GPIO5: now also J5.4 (Pin_4)
- removed net GPIO: J5.1 (Pin_1), J5.2 (Pin_2), J5.3 (Pin_3), J5.4 (Pin_4)
- new net GPIO3: J5.2 (Pin_2), U7.3 (LRCLK2)
Other:
- moved on the sheet: J5, J6

Commit message: began routing
Connections:
- net +3V3: now also U7.3.3V_2 (3.3V__1); no longer U7.3.3V_1 (3.3V)
- net SCK: no longer U7.13 (SCK)
- net SPI_SCK: now also U7.13 (SCK)
- net V_BUCK: now also JP1.3 (B); no longer JP1.1 (A)
- net V_LDO: now also JP1.1 (A); no longer JP1.3 (B)
- net GPIO24: now reaches U7.24 (A10)
- net GPIO24: now also J5.4 (Pin_4)
- net GPIO25: now reaches U7.25 (A11)
- net GPIO25: now also J5.3 (Pin_3)
- net GPIO26: now reaches U7.26 (A12)
- net GPIO26: now also J5.2 (Pin_2)
- net GPIO27: now reaches U7.27 (A13)
- net GPIO27: now also J5.1 (Pin_1)
- net GPIO2: no longer names the net of U7.2 (OUT2)
- net GPIO2: no longer J5.1 (Pin_1)
- net GPIO3: no longer names the net of U7.3 (LRCLK2)
- net GPIO3: no longer J5.2 (Pin_2)
- net GPIO4: no longer names the net of U7.4 (BCLK2)
- net GPIO4: no longer J5.3 (Pin_3)
- net GPIO5: no longer names the net of U7.5 (IN2)
- net GPIO5: no longer J5.4 (Pin_4)
Other:
- moved on the sheet: C14, C15, C16, H1, H2, H3, H4, JP2, U8

Commit message: updates
Connections:
- net MISO is gone; now on net SPI_MISO: U1.7 (SO), U2.7 (SO), U3.7 (SO)
- net SCK is gone; now on net SPI_SCK: U1.5 (SCK), U2.5 (SCK), U3.5 (SCK)
- net T1_CS: now also U7.22 (A8); no longer U7.20 (A6)
- net T3_CS: now also U7.20 (A6); no longer U7.22 (A8)
Other:
- moved on the sheet: C5, C6, C7
Changed lines of the file:
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@@
 		)
 	)
-	(hierarchical_label "SCK"
+	(hierarchical_label "SPI_SCK"
 		(shape input)
 		(at 334.01 35.56 0)
@@
 		)
 	)
-	(hierarchical_label "SCK"
+	(hierarchical_label "SPI_SCK"
 		(shape input)
 		(at 334.01 106.68 0)
@@
 		)
 	)
-	(hierarchical_label "SCK"
+	(hierarchical_label "SPI_SCK"
 		(shape input)
 		(at 334.01 71.12 0)
@@
 		)
 	)
-	(hierarchical_label "MISO"
+	(hierarchical_label "SPI_MISO"
 		(shape output)
 		(at 334.01 38.1 0)
@@
 		)
 	)
-	(hierarchical_label "MISO"
+	(hierarchical_label "SPI_MISO"
 		(shape output)
 		(at 334.01 73.66 0)
@@
 		)
 	)
-	(hierarchical_label "MISO"
+	(hierarchical_label "T1_CS"
+		(shape input)
+		(at 224.79 119.38 180)
+		(fields_autoplaced yes)
+		(effects
+			(font
+				(size 1.27 1.27)
+			)
+			(justify right)
+		)
+	)
+	(hierarchical_label "SPI_MISO"
 		(shape output)
 		(at 334.01 109.22 0)
@@
 		)
 	)
-	(hierarchical_label "T1_CS"
-		(shape input)
-		(at 224.79 114.3 180)
-		(fields_autoplaced yes)
-		(effects
-			(font
-				(size 1.27 1.27)
-			)
-			(justify right)
-		)
-	)
 	(hierarchical_label "DS18_TEMP"
 		(shape output)
@@
 		)
 	)
-	(hierarchical_label "T3_CS"
-		(shape input)
-		(at 224.79 119.38 180)
-		(fields_autoplaced yes)
-		(effects
-			(font
-				(size 1.27 1.27)
-			)
-			(justify right)
-		)
-	)
 	(hierarchical_label "T2_CS"
 		(shape output)
@@
 		)
 	)
+	(hierarchical_label "T3_CS"
+		(shape input)
+		(at 224.79 114.3 180)
+		(fields_autoplaced yes)
+		(effects
+			(font
+				(size 1.27 1.27)
+			)
+			(justify right)
+		)
+	)
 	(hierarchical_label "T3"
 		(shape input)
@@
 	(symbol
 		(lib_id "power:+3V3")
-		(at 345.44 35.56 0)
+		(at 349.25 34.29 0)
 		(unit 1)
 		(exclude_from_sim no)
@@
 		(fields_autoplaced yes)
 		(property "Reference" "#PWR010"
-			(at 345.44 39.37 0)
+			(at 349.25 38.1 0)
 			(effects
 				(font
@@
 		)
 		(property "Value" "+3V3"
-			(at 345.44 30.48 0)
+			(at 349.25 29.21 0)
 			(effects
 				(font
@@
 		)
 		(property "Footprint" ""
-			(at 345.44 35.56 0)
+			(at 349.25 34.29 0)
 			(effects
 				(font
@@
 		)
 		(property "Datasheet" ""
-			(at 345.44 35.56 0)
+			(at 349.25 34.29 0)
 			(effects
 				(font
@@
 		)
 		(property "Description" "Power symbol creates a global label with name \"+3V3\""
-			(at 345.44 35.56 0)
+			(at 349.25 34.29 0)
 			(effects
 				(font
@@
 	(symbol
 		(lib_id "power:+3V3")
-		(at 346.71 107.95 0)
+		(at 350.52 106.68 0)
 		(unit 1)
 		(exclude_from_sim no)
@@
 		(fields_autoplaced yes)
 		(property "Reference" "#PWR014"
-			(at 346.71 111.76 0)
+			(at 350.52 110.49 0)
 			(effects
 				(font
@@
 		)
 		(property "Value" "+3V3"
-			(at 346.71 102.87 0)
+			(at 350.52 101.6 0)
 			(effects
 				(font
@@
 		)
 		(property "Footprint" ""
-			(at 346.71 107.95 0)
+			(at 350.52 106.68 0)
 			(effects
 				(font
@@
 		)
 		(property "Datasheet" ""
-			(at 346.71 107.95 0)
+			(at 350.52 106.68 0)
 			(effects
 				(font
@@
 		)
 		(property "Description" "Power symbol creates a global label with name \"+3V3\""
-			(at 346.71 107.95 0)
+			(at 350.52 106.68 0)
 			(effects
 				(font
@@
 	(symbol
 		(lib_id "power:+3V3")
-		(at 345.44 71.12 0)
+		(at 349.25 69.85 0)
 		(unit 1)
 		(exclude_from_sim no)
@@
 		(fields_autoplaced yes)
 		(property "Reference" "#PWR012"
-			(at 345.44 74.93 0)
+			(at 349.25 73.66 0)
 			(effects
 				(font
@@
 		)
 		(property "Value" "+3V3"
-			(at 345.44 66.04 0)
+			(at 349.25 64.77 0)
 			(effects
 				(font
@@
 		)
 		(property "Footprint" ""
-			(at 345.44 71.12 0)
+			(at 349.25 69.85 0)
 			(effects
 				(font
@@
 		)
 		(property "Datasheet" ""
-			(at 345.44 71.12 0)
+			(at 349.25 69.85 0)
 			(effects
 				(font
@@
 		)
 		(property "Description" "Power symbol creates a global label with name \"+3V3\""
-			(at 345.44 71.12 0)
+			(at 349.25 69.85 0)
 			(effects
 				(font
@@
 	(symbol
 		(lib_id "power:GND")
-		(at 346.71 115.57 0)
+		(at 350.52 114.3 0)
 		(unit 1)
 		(exclude_from_sim no)
@@
 		(fields_autoplaced yes)
 		(property "Reference" "#PWR015"
-			(at 346.71 121.92 0)
+			(at 350.52 120.65 0)
 			(effects
 				(font
@@
 		)
 		(property "Value" "GND"
-			(at 346.71 120.65 0)
+			(at 350.52 119.38 0)
 			(effects
 				(font
@@
 		)
 		(property "Footprint" ""
-			(at 346.71 115.57 0)
+			(at 350.52 114.3 0)
 			(effects
 				(font
@@
 		)
 		(property "Datasheet" ""
-			(at 346.71 115.57 0)
+			(at 350.52 114.3 0)
 			(effects
 				(font
@@
 		)
 		(property "Description" "Power symbol creates a global label with name \"GND\" , ground"
-			(at 346.71 115.57 0)
+			(at 350.52 114.3 0)
 			(effects
 				(font
@@
 	(symbol
 		(lib_id "Device:C")
-		(at 345.44 39.37 0)
+		(at 349.25 38.1 0)
 		(unit 1)
 		(exclude_from_sim no)
@@
 		(fields_autoplaced yes)
 		(property "Reference" "C5"
-			(at 349.25 38.0999 0)
+			(at 353.06 36.8299 0)
 			(effects
 				(font
@@
 		)
 		(property "Value" "0.1uF"
-			(at 349.25 40.6399 0)
+			(at 353.06 39.3699 0)
 			(effects
 				(font
@@
 		)
 		(property "Footprint" "Capacitor_SMD:C_0805_2012Metric_Pad1.18x1.45mm_HandSolder"
-			(at 346.4052 43.18 0)
+			(at 350.2152 41.91 0)
 			(effects
 				(font
@@
 		)
 		(property "Datasheet" "~"
-			(at 345.44 39.37 0)
+			(at 349.25 38.1 0)
 			(effects
 				(font
@@
 		)
 		(property "Description" "Unpolarized capacitor"
-			(at 345.44 39.37 0)
+			(at 349.25 38.1 0)
 			(effects
 				(font
@@
 	(symbol
 		(lib_id "power:GND")
-		(at 345.44 78.74 0)
+		(at 349.25 77.47 0)
 		(unit 1)
 		(exclude_from_sim no)
@@
 		(fields_autoplaced yes)
 		(property "Reference" "#PWR013"
-			(at 345.44 85.09 0)
+			(at 349.25 83.82 0)
 			(effects
 				(font
@@
 		)
 		(property "Value" "GND"
-			(at 345.44 83.82 0)
+			(at 349.25 82.55 0)
 			(effects
 				(font
@@
 		)
 		(property "Footprint" ""
-			(at 345.44 78.74 0)
+			(at 349.25 77.47 0)
 			(effects
 				(font
@@
 		)
 		(property "Datasheet" ""
-			(at 345.44 78.74 0)
+			(at 349.25 77.47 0)
 			(effects
 				(font
@@
 		)
 		(property "Description" "Power symbol creates a global label with name \"GND\" , ground"
-			(at 345.44 78.74 0)
+			(at 349.25 77.47 0)
 			(effects
 				(font
@@
 	(symbol
 		(lib_id "Device:C")
-		(at 345.44 74.93 0)
+		(at 349.25 73.66 0)
 		(unit 1)
 		(exclude_from_sim no)
@@
 		(fields_autoplaced yes)
 		(property "Reference" "C6"
-			(at 349.25 73.6599 0)
+			(at 353.06 72.3899 0)
 			(effects
 				(font
@@
 		)
 		(property "Value" "0.1uF"
-			(at 349.25 76.1999 0)
+			(at 353.06 74.9299 0)
 			(effects
 				(font
@@
 		)
 		(property "Footprint" "Capacitor_SMD:C_0805_2012Metric_Pad1.18x1.45mm_HandSolder"
-			(at 346.4052 78.74 0)
+			(at 350.2152 77.47 0)
 			(effects
 				(font
@@
 		)
 		(property "Datasheet" "~"
-			(at 345.44 74.93 0)
+			(at 349.25 73.66 0)
 			(effects
 				(font
@@
 		)
 		(property "Description" "Unpolarized capacitor"
-			(at 345.44 74.93 0)
+			(at 349.25 73.66 0)
 			(effects
 				(font
@@
 	(symbol
 		(lib_id "power:GND")
-		(at 345.44 43.18 0)
+		(at 349.25 41.91 0)
 		(unit 1)
 		(exclude_from_sim no)
@@
 		(fields_autoplaced yes)
 		(property "Reference" "#PWR011"
-			(at 345.44 49.53 0)
+			(at 349.25 48.26 0)
 			(effects
 				(font
@@
 		)
 		(property "Value" "GND"
-			(at 345.44 48.26 0)
+			(at 349.25 46.99 0)
 			(effects
 				(font
@@
 		)
 		(property "Footprint" ""
-			(at 345.44 43.18 0)
+			(at 349.25 41.91 0)
 			(effects
 				(font
@@
 		)
 		(property "Datasheet" ""
-			(at 345.44 43.18 0)
+			(at 349.25 41.91 0)
 			(effects
 				(font
@@
 		)
 		(property "Description" "Power symbol creates a global label with name \"GND\" , ground"
-			(at 345.44 43.18 0)
+			(at 349.25 41.91 0)
 			(effects
 				(font
@@
 	(symbol
 		(lib_id "Device:C")
-		(at 346.71 111.76 0)
+		(at 350.52 110.49 0)
 		(unit 1)
 		(exclude_from_sim no)
@@
 		(fields_autoplaced yes)
 		(property "Reference" "C7"
-			(at 350.52 110.4899 0)
+			(at 354.33 109.2199 0)
 			(effects
 				(font
@@
 		)
 		(property "Value" "0.1uF"
-			(at 350.52 113.0299 0)
+			(at 354.33 111.7599 0)
 			(effects
 				(font
@@
 		)
 		(property "Footprint" "Capacitor_SMD:C_0805_2012Metric_Pad1.18x1.45mm_HandSolder"
-			(at 347.6752 115.57 0)
+			(at 351.4852 114.3 0)
 			(effects
 				(font
@@
 		)
 		(property "Datasheet" "~"
-			(at 346.71 111.76 0)
+			(at 350.52 110.49 0)
 			(effects
 				(font
@@
 		)
 		(property "Description" "Unpolarized capacitor"
-			(at 346.71 111.76 0)
+			(at 350.52 110.49 0)
 			(effects
 				(font

Commit message: rework
Parts:
- added M1: Fan_4pin, Connector:FanPinHeader_1x04_P2.54mm_Vertical, symbol Motor:Fan_4pin
- J2: footprint Connector_AMASS:AMASS_XT60-M_1x02_P7.20mm_Vertical -> Connector_AMASS:AMASS_XT60IPW-M_1x03_P7.20mm_Horizontal
Connections:
- net +5V: now also M1.2 (+)
- net +BATT: now also J2.2 (+); no longer J2.1 (+)
- net GND: now also J2.1 (-), M1.1 (-); no longer J2.2 (-)
- net FAN_PWM: now reaches U7.33 (MCLK2)
- net FAN_PWM: now also M1.4 (PWM)
- net FAN_TACHO: now reaches U7.34 (RX8)
- net FAN_TACHO: now also M1.3 (Tacho)
