File: payload/pcb/IREC_HeatTransfer_Payload/IREC_HeatTransfer_Payload.kicad_pcb (KiCad board)
At the start: 2 copper layers, 63.5 x 101.6 mm, 53 parts, among them J1 Screw_Terminal_01x06, J2 XT60PW-M, J3 Screw_Terminal_01x06, J4 POWER, J5 GPIO, J6 SPI, J7 I2C, J9 Serial, U1 MAX31855KASA, U2 MAX31855KASA, U3 MAX31855KASA, U4 AP63357, U5 DS18B20, U6 NJM7805SDL1-TE1, U7 DEV-16771, U8 MPXV7002DP

Commit message: rework
Parts:
- added M1: Fan_4pin, Connector:FanPinHeader_1x04_P2.54mm_Vertical, F.Cu at (209.4, 59.7)
- J2: footprint Connector_AMASS:AMASS_XT60-M_1x02_P7.20mm_Vertical -> Connector_AMASS:AMASS_XT60IPW-M_1x03_P7.20mm_Horizontal
- moved J2 15.6 mm to (170.0, 63.1), turned to 0 degrees
- moved U6 15.5 mm to (177.0, 92.3)
- moved D1 14.4 mm to (170.2, 74.9)
- moved C11 14.4 mm to (167.3, 70.6)
- moved L1 14.4 mm to (161.4, 73.4)
- moved R4 14.4 mm to (158.7, 61.5)
- moved U4 14.4 mm to (159.1, 66.9)
- moved C12 14.4 mm to (167.3, 75.2)
- moved R5 14.4 mm to (155.6, 64.7)
- moved C4 14.4 mm to (162.5, 66.8)
- moved C9 14.4 mm to (158.8, 63.7)
- moved C8 14.4 mm to (155.6, 69.3)
- moved JP1 10.7 mm to (169.9, 86.6), turned to 180 degrees
- moved R7 10.1 mm to (183.1, 80.5), turned to -90 degrees
- moved R1 9.52 mm to (172.5, 80.5), turned to -90 degrees
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Connections:
- J2 pad 1: +BATT -> GND
- J2 pad 2: GND -> +BATT
- U7 pad 33: unconnected-(U7-MCLK2-Pad33) -> /FAN_PWM
- U7 pad 34: unconnected-(U7-RX8-Pad34) -> /FAN_TACHO
Routing:
- net /PITOT: track 42.3 -> 0.00 mm, vias 1 -> 0
- net /VBAT_SENSE: track 32.1 -> 2.52 mm, vias 1 -> 0
- net V_BUCK: track 29.7 -> 1.08 mm, vias 2 -> 1
- net +BATT: track 19.1 -> 43.7 mm
- net +5V: track 109.2 -> 89.2 mm, vias 3 -> 5
- net VCC: track 42.7 -> 25.7 mm
- net Net-(D1-PadA): track 8.27 -> 0.00 mm, vias 1 -> 0
- net V_LDO: track 15.5 -> 8.75 mm
- net /GPIO24: track 25.3 -> 24.3 mm
- net GND: track 7.89 -> 7.59 mm, vias 71 -> 68
Other:
- board text added: "Heat Flow Sensor Board"
- board text added: "MAX REC 7.4V"
- board text removed: "TC / Pitot Board"

Commit message: upd
Parts:
- removed M1: Fan_4pin, Connector:FanPinHeader_1x04_P2.54mm_Vertical
- added C11: 0.33uF, Capacitor_SMD:C_0805_2012Metric_Pad1.18x1.45mm_HandSolder, B.Cu at (188.2, 48.5)
- added C12: 0.1uF, Capacitor_SMD:C_0805_2012Metric_Pad1.18x1.45mm_HandSolder, B.Cu at (200.9, 48.5)
- added J9: FAN, Connector_PinHeader_2.54mm:PinHeader_1x02_P2.54mm_Vertical, F.Cu at (211.3, 62.0)
- added Q1: 2N7002K, Package_TO_SOT_SMD:SOT-23, B.Cu at (206.9, 64.5)
- added U6: L78M12CDT-TR, CustomFootprintLib:VREG_L78M12CDT-TR, B.Cu at (194.6, 52.7)
- C1: renamed from C4; value 10uF -> 0.33uF; moved to B.Cu
- C2: renamed from C10; value 0.33uF -> 10uF; moved to F.Cu
- JP1: moved to B.Cu
- moved C1 18.8 mm to (175.3, 80.5), turned to 90 degrees
- moved C2 18.7 mm to (162.3, 66.8), turned to -90 degrees
- moved JP1 0.22 mm to (169.7, 86.6)
- turned R8 to 90 degrees
- renumbered C12 to C10, C1 to C13, C2 to C14, C3 to C15, C5 to C16, C6 to C17, C7 to C18, C8 to C6, C9 to C7, C13 to C8, C11 to C9, J4 to J1, J7 to J2, J9 to J3, J6 to J4, J2 to J6, J3 to J7, J1 to J8, R6 to R4, R4 to R5, R5 to R6, R7 to R8, R8 to R9, TP3 to TP1, TP1 to TP2, TP2 to TP3, U5 to U1, U8 to U2, U6 to U3, U7 to U5, U1 to U7, U2 to U8, U3 to U9
Connections:
- net +BATT renamed /+BATT
- net VCC renamed /+VCC
- C1 pad 1: V_BUCK -> 5V_LDO
- C2 pad 1: V_LDO -> 5V_BUCK
- JP1 pad 1: V_LDO -> 5V_LDO
- JP1 pad 3: V_BUCK -> 5V_BUCK
- U3 pad 1: V_LDO -> 5V_LDO
- U4 pad 1: V_BUCK -> 5V_BUCK
- U4 pad 2: V_BUCK -> 5V_BUCK
- U5 pad 14: /DS18_TEMP -> /FAN
- U5 pad 15: /VBAT_SENSE -> /DS18_TEMP
- U5 pad 16: /PITOT -> /VBAT_SENSE
- U5 pad 17: unconnected-(U7-A3-Pad17) -> /PITOT
- U5 pad 33: /FAN_PWM -> unconnected-(U5-MCLK2-Pad33)
- U5 pad 34: /FAN_TACHO -> unconnected-(U5-RX8-Pad34)
Routing:
- net /FAN: track 0.00 -> 63.2 mm
- net /+VCC: track 25.7 -> 87.2 mm
- net /PITOT: track 0.00 -> 52.2 mm, vias 0 -> 1
- net 5V_BUCK: track 0.00 -> 32.4 mm, vias 0 -> 1
- net /VBAT_SENSE: track 2.52 -> 31.5 mm, vias 0 -> 2
- net /+12V: track 0.00 -> 21.7 mm
- net +5V: track 89.2 -> 101.6 mm
- net 5V_LDO: track 0.00 -> 8.84 mm
- net V_LDO: track 8.75 -> 0.00 mm, vias 1 -> 0
- net Net-(D1-PadA): track 0.00 -> 6.51 mm, vias 0 -> 1
- net /DS18_TEMP: track 32.0 -> 36.2 mm, vias 0 -> 1
- net Net-(J9-Pin_2): track 0.00 -> 3.38 mm
- net GND: track 7.59 -> 4.39 mm
- net V_BUCK: track 1.08 -> 0.00 mm, vias 1 -> 0
- added copper zone on B.Cu, net 5V_BUCK
- added copper zone on F.Cu, net 5V_BUCK
- removed copper zone on B.Cu, net V_BUCK
- removed copper zone on F.Cu, net V_BUCK
Other:
- board text added: "+5V"
- board text added: "FAN+"
- board text added: "FAN-"
- board text added: "PSU 12.6V"
- board text removed: "MAX REC 7.4V"
