File: payload/boards/VULCAN/VULCAN.kicad_sch (KiCad schematic)
At the start: 59 parts, among them J1 POWER, J2 I2C, J3 Serial, J4 SPI, J5 GPIO, J6 XT60PW-M, J7 Screw_Terminal_01x06, J8 Screw_Terminal_01x06, J9 FAN, Q1 2N7002K, U1 DS18B20, U2 MPXV7002DP, U3 NJM7805SDL1-TE1, U4 AP63357, U5 DEV-16771, U6 L78M12CDT-TR, U7 MAX31855KASA, U8 MAX31855KASA, U9 MAX31855KASA

Commit message: upd
Parts:
- removed C11: 0.33uF, Capacitor_SMD:C_0805_2012Metric_Pad1.18x1.45mm_HandSolder, symbol Device:C
- removed C12: 0.1uF, Capacitor_SMD:C_0805_2012Metric_Pad1.18x1.45mm_HandSolder, symbol Device:C
- removed U6: L78M12CDT-TR, CustomFootprintLib:VREG_L78M12CDT-TR, symbol CustomComponents:L78M12CDT-TR
- added D3: OSRAM_LSR976-NR-1, Skyhawkson_Footprints:OSRAM_0805, symbol Skyhawkson-LEDs and Optoelectronics:OSRAM_LSR976-NR-1
- added R8: R, Resistor_SMD:R_0805_2012Metric_Pad1.20x1.40mm_HandSolder, symbol Device:R
- J9: footprint Connector_PinHeader_2.54mm:PinHeader_1x02_P2.54mm_Vertical -> Molex_KK-254_AE-6410-02A_1x02_P2.54mm_Vertical
- renumbered C13 to C11, C14 to C12, C15 to C13, C16 to C14, C17 to C15, C18 to C16, R9 to R10, R8 to R9, TP2 to TP1, TP1 to TP2, U3 to U2, U2 to U3, U7 to U6, U8 to U7, U9 to U8
Connections:
- net +VCC is gone; now on net +12V: J1.1 (Pin_1), J7.4 (Pin_4), JP1.2 (C), R9.1, TP2.1
- net GND: now also D3.C, R8.1
- new net: D3.A, R8.2
Other:
- note removed: "12V Voltage Regulator"
- note removed: "L78M12CDT"

Commit message: updates
Parts:
- added IC1: LT1001CS8#PBF, Amplifier_Operational_Analog:Analog_LT1001_CS8, symbol Amplifier_Operational_Analog:LT1001CS8#PBF
- added JP3: Jumper_2_Open, Jumper:SolderJumper-2_P1.3mm_Open_RoundedPad1.0x1.5mm, symbol Jumper:Jumper_2_Open
- added R11, R12: 1K, Resistor_SMD:R_0805_2012Metric_Pad1.20x1.40mm_HandSolder, symbol Device:R_US
- added R13, R14: 5K, Resistor_SMD:R_0805_2012Metric_Pad1.20x1.40mm_HandSolder, symbol Device:R_US
- added R_Shunt1: 0.1, Package_TO_SOT_SMD:TO-263-2_TabPin1, symbol Device:R_US
Connections:
- net +12V: now also JP3.1 (A), R12.1, R_Shunt1.1; no longer J7.4 (Pin_4)
- net GND: now also IC1.4 (V-), R13.1
- net +BATT renamed +BATT_RAW
- new net: IC1.2 (-IN), R12.2, R14.2
- new net: IC1.3 (+IN), R11.2, R13.2
- new net +12V_RAW: IC1.7 (V+), J7.4 (Pin_4), JP3.2 (B), R11.1, R_Shunt1.2
- new net VBAT_CURRENT_SENSE: IC1.6 (OUT), R14.1
- no-connect marks 40 -> 43
Other:
- note added: "!!!WARNING: Using incorrect batteries or power sources may damage electronics!!!"
- note added: "Connect jumper to bypass shunt resistor in event of failure."
- note added: "Current Sensing Shunt Resistor"
- note added: "Grid Size: 2.54mm"
- note added: "PFS35-0R1F1"
- note added: "Shunt Resistor: 35W MAX"
- note added: "To-Do - Add current sensing?"

Commit message: updates
Parts:
- D3: Color RED -> GREEN
Other:
- note added: "To-Do - Add current sensing? (size down shunt?)"
- note removed: "To-Do - Add current sensing?"
Changed lines of the file:
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@@
 		)
 	)
-	(text "To-Do\n- Add current sensing?"
+	(text "To-Do\n- Add current sensing? (size down shunt?)"
 		(exclude_from_sim no)
 		(at 422.656 164.592 0)
@@
 		(dnp no)
 		(property "Reference" "D3"
-			(at 193.548 157.48 0)
+			(at 191.516 157.226 0)
 			(effects
 				(font
@@
 			)
 		)
-		(property "Color" "RED"
-			(at 191.008 156.464 0)
+		(property "Color" "GREEN"
+			(at 193.548 153.67 0)
 			(effects
 				(font

Commit message: updates
Parts:
- removed U2: NJM7805SDL1-TE1, CustomFootprintLib:TO-252-3-L1_NMD, symbol CustomComponents:NJM7805SDL1-TE1
- added U2: AZ1117IH-5.0TRG1, CustomFootprintLib:SOT223-5_DIO, symbol CustomComponents:AZ1117IH-5.0TRG1
- BT1: footprint Battery:BatteryHolder_Keystone_3002_1x2032 -> Battery:BatteryHolder_Keystone_1060_1x2032
- C1: value 0.33uF -> 22uF
- C8: value 0.1uF -> 10uF
- R_Shunt1: value 0.1 -> 0.05; footprint Package_TO_SOT_SMD:TO-263-2_TabPin1 -> Resistor_SMD:R_2816_7142Metric_Pad3.20x4.45mm_HandSolder
- TP1, TP2, TP3: now left out of the parts list
Connections:
- net +5V: now also C1.1, U2.2 (OUTPUT); no longer C8.1
- net 5V_LDO: now also C8.1, U2.3 (INPUT); no longer C1.1
- net GND: now also U2.1 (ADJ/GND)
- no-connect marks 43 -> 44
Other:
- note added: "1A IOUT MAX 15V VIN MAX 5V VOUT"
- note added: "AZ1117IH-5.0TRG1"
- note removed: "NJM7805SDL1-TE1"

Commit message: upd
Parts:
- R9: value 200k -> 300k
Connections:
- net DS18_TEMP: now also U5.40 (A16); no longer U5.15 (A1)
- net VBAT_CURRENT_SENSE: now also U5.41 (A17)
- no-connect marks 44 -> 41
Other:
- note added: "ATMEGA328 ADC reads 0-3.3V"
- note added: "Teensy RTC"
- note removed: "To-Do - Add current sensing? (size down shunt?)"
- moved on the sheet: BT1, C11, C12, C13, C14, C15, C16, C3, C4, C5, D3, H1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

Commit message: updates
1-wire sensor
Parts:
- removed C11, C12, C13: 100n, Capacitor_SMD:C_0805_2012Metric_Pad1.18x1.45mm_HandSolder, symbol Device:C
- removed C14, C15, C16: 0.1uF, Capacitor_SMD:C_0805_2012Metric_Pad1.18x1.45mm_HandSolder, symbol Device:C
- removed D2: OSRAM_LGR971-KN-1, Skyhawkson_Footprints:OSRAM_0805, symbol Skyhawkson-LEDs and Optoelectronics:OSRAM_LGR971-KN-1
- removed R8: R, Resistor_SMD:R_0805_2012Metric_Pad1.20x1.40mm_HandSolder, symbol Device:R
- removed U6, U7, U8: MAX31855KASA, Package_SO:SOIC-8_3.9x4.9mm_P1.27mm, symbol Sensor_Temperature:MAX31855KASA
- added C6, C7, C8: 0.1uF, Capacitor_SMD:C_0805_2012Metric_Pad1.18x1.45mm_HandSolder, symbol Device:C
- added D2: CMD17-21VGD/TR8, Skyhawkson_Footprints:OSRAM_0805, symbol Skyhawkson-LEDs and Optoelectronics:OSRAM_LSR976-NR-1
- added FB1, FB2, FB3, FB4, FB5, FB6: Ferrite_Bead, PCM_Ferrite_SMD_AKL:Ferrite_0805_2012Metric_Pad1.05x1.20mm_BigPads, symbol PCM_Device_AKL:Ferrite_Bead
- added R10: 500, Resistor_SMD:R_0805_2012Metric_Pad1.20x1.40mm_HandSolder, symbol Device:R
- added R17: 4.7k, Resistor_SMD:R_0805_2012Metric_Pad1.20x1.40mm_HandSolder, symbol Device:R
- added R7, R9: R, Resistor_SMD:R_0805_2012Metric_Pad1.20x1.40mm_HandSolder, symbol Device:R
- added U6, U7, U8: MAX31850KATB+T, CustomFootprintLib:SON50P300X400X80-11N, symbol CustomComponents:MAX31850KATB+T
- C11: renamed from C3; footprint (none) -> Capacitor_SMD:C_0805_2012Metric_Pad1.18x1.45mm_HandSolder
- C12: renamed from C4; footprint (none) -> Capacitor_SMD:C_0805_2012Metric_Pad1.18x1.45mm_HandSolder
- C13: renamed from C5; footprint (none) -> Capacitor_SMD:C_0805_2012Metric_Pad1.18x1.45mm_HandSolder
- D3: value OSRAM_LSR976-NR-1 -> CMD17-21VGD/TR8
- J9: footprint Molex_KK-254_AE-6410-02A_1x02_P2.54mm_Vertical -> CustomFootprintLib:Molex_KK-254_AE-6410-02A_1x02_P2.54mm_Vertical
- R1: value R -> 150
- R2: value R -> 68
- R8: renamed from R7; footprint (none) -> Resistor_SMD:R_0805_2012Metric_Pad1.20x1.40mm_HandSolder
- renumbered C6 to C3, C7 to C4, C8 to C5, R9 to R11, R10 to R12, R11 to R13, R12 to R14, R13 to R15, R14 to R16, U4 to U3, U3 to U4
Connections:
- net +12V: now also R10.1
- net +3V3: now also R17.2, R7.1, R9.1, U6.4 (VDD), U7.4 (VDD), U8.4 (VDD)
- net GND: now also D2.C, U6.1 (GND), U7.1 (GND), U8.1 (GND); no longer D3.C
- net I2C_SCL: now also R9.2
- net I2C_SDA: now also R7.2
- net T-: now also C6.2, C7.2, C8.2, FB2.2, FB4.2, FB6.2, U6.2 (T-), U7.2 (T-), U8.2 (T-); no longer J8.2 (Pin_2), J8.4 (Pin_4), J8.6 (Pin_6)
- net T1: now also C6.1, FB1.2, U6.3 (T+); no longer J8.1 (Pin_1)
- net T2: now also C8.1, FB3.2, U7.3 (T+); no longer J8.3 (Pin_3)
- net T3: now also C7.1, FB5.2, U8.3 (T+); no longer J8.5 (Pin_5)
- net at R2.1: now also D2.A
- net at D3.A: now also R10.2
- net at J9.2 (Pin_2), Q1.3 (D): now also D3.C
- net T1_CS: no longer names the net of U5.22 (A8)
- net T2_CS: no longer names the net of U5.21 (A7)
- net T3_CS renamed TC_DATA
- net TC_DATA: now also R17.1, U6.5 (DQ), U7.5 (DQ), U8.5 (DQ)
- new net: FB6.1, J8.6 (Pin_6)
- new net: FB2.1, J8.2 (Pin_2)
- new net: FB4.1, J8.4 (Pin_4)
- new net: FB1.1, J8.1 (Pin_1)
- new net: FB5.1, J8.5 (Pin_5)
- new net: FB3.1, J8.3 (Pin_3)
- no-connect marks 41 -> 60
Other:
- note added: "Pull-Up Resistors (Opt.)"
- note added: "Thermocouples (Type-K)"
- moved on the sheet: BT1, C1, C11, C12, C13, C5, D1, H1, H2, H3, H4, IC1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

Commit message: updates
Parts:
- BT1: Purchase (none) -> https://www.digikey.com/en/products/detail/keystone-electro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
- D1: value OSRAM_LSR976-NR-1 -> CMD17-21VRD/TR8; Purchase (none) -> https://www.digikey.com/en/products/detail/visual-communica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
- D2, D3: Purchase (none) -> https://www.digikey.com/en/products/detail/visual-communica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
- IC1, U6, U7, U8: Purchase (none) -> https://www.digikey.com/en/products/detail/analog-devices-i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
- J7, J8: Purchase (none) -> https://www.digikey.com/en/products/detail/on-shore-technol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
- J9: Purchase (none) -> https://www.digikey.com/en/products/detail/molex/0022272021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
- L1: Purchase (none) -> https://www.digikey.com/en/products/detail/bourns-inc/SRN80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
- Q1: Purchase (none) -> https://www.digikey.com/en/products/detail/onsemi/2N7002K/2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
- U1: Purchase (none) -> https://www.digikey.com/en/products/detail/umw/DS18B20/1670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
- U2, U3: Purchase (none) -> https://www.digikey.com/en/products/detail/diodes-incorpora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
- U4: Purchase (none) -> https://www.digikey.com/en/products/detail/nxp-usa-inc/mpxv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
- U5: Purchase (none) -> https://www.sparkfun.com/products/16996
Connections:
- no-connect marks 60 -> 62

Commit message: rework
boost converter stuff
Parts:
- removed C10, C9: 22uF, Capacitor_SMD:C_0805_2012Metric_Pad1.18x1.45mm_HandSolder, symbol Device:C
- removed C2: 10uF, Capacitor_SMD:C_0805_2012Metric_Pad1.18x1.45mm_HandSolder, symbol Device:C
- removed C3: 0.1u, Capacitor_SMD:C_0805_2012Metric_Pad1.18x1.45mm_HandSolder, symbol Device:C
- removed C4: 47pF, Capacitor_SMD:C_0805_2012Metric_Pad1.18x1.45mm_HandSolder, symbol Device:C
- removed D3: CMD17-21VGD/TR8, Skyhawkson_Footprints:OSRAM_0805, symbol Skyhawkson-LEDs and Optoelectronics:OSRAM_LSR976-NR-1
- removed J9: FAN, CustomFootprintLib:Molex_KK-254_AE-6410-02A_1x02_P2.54mm_Vertical, symbol Connector_Generic:Conn_01x02
- removed JP1: Jumper_3_Open, Jumper:SolderJumper-3_P1.3mm_Open_RoundedPad1.0x1.5mm, symbol Jumper:Jumper_3_Open
- removed L1: 6.8uH, CustomFootprintLib:IND_SRN8040TA-6R8M, symbol Device:L
- removed Q1: 2N7002K, Package_TO_SOT_SMD:SOT-23, symbol Transistor_FET:2N7002K
- removed R5: 220k, Resistor_SMD:R_0805_2012Metric_Pad1.20x1.40mm_HandSolder, symbol Device:R
- removed R6: 41.2k, Resistor_SMD:R_0805_2012Metric_Pad1.20x1.40mm_HandSolder, symbol Device:R
- removed TP2: VIN, TestPoint:TestPoint_Pad_D1.0mm, symbol Connector:TestPoint
- removed TP3: +5V, TestPoint:TestPoint_Pad_D1.0mm, symbol Connector:TestPoint
- removed U2: AZ1117IH-5.0TRG1, CustomFootprintLib:SOT223-5_DIO, symbol CustomComponents:AZ1117IH-5.0TRG1
- removed U3: AP63357, CustomFootprintLib:AP63356 (V-DFN3020-13), symbol CustomComponents:AP63357_(SparkFun_Buck_Regulator_5V)
- added C14, C15: 10uF, Capacitor_SMD:C_0805_2012Metric_Pad1.18x1.45mm_HandSolder, symbol Device:C
- added F1: LF_0494003, Skyhawkson_Footprints:LF_0494_(0603), symbol Skyhawkson-Miscellaneous:LF_0494003
- added L2: 2.2uH, symbol Device:L
- added R18: 2M, Resistor_SMD:R_0805_2012Metric_Pad1.20x1.40mm_HandSolder, symbol Device:R
- added R19: 220k, Resistor_SMD:R_0805_2012Metric_Pad1.20x1.40mm_HandSolder, symbol Device:R
- added U2: TPS61200DRC, Package_SON:Texas_S-PVSON-N10_ThermalVias, symbol Regulator_Switching:TPS61200DRC
- C1: value 22uF -> 10uF
- C5: value 10uF -> 1uF
- R10: value 500 -> 2M
- R8: value 470 -> 220k
Connections:
- net +12V: no longer JP3.1 (A), R10.1, R11.1, R14.1, R_Shunt1.1
- net +3V3: now also U7.6 (AD0), U8.7 (AD1)
- net +5V: now also R10.1, C14.2, C15.2, U2.2 (VOUT); no longer C1.1
- net FAN: no longer R8.2
- net GND: now also C1.1, R8.2, U6.6 (AD0), U6.7 (AD1), U6.8 (AD2), U6.9 (AD3), U7.7 (AD1), U7.8 (AD2), U7.9 (AD3), U8.6 (AD0), U8.8 (AD2), U8.9 (AD3), C14.1, C15.1, R18.2, R19.1, U2.11 (PAD), U2.4 (PGND), U2.5 (VIN), U2.6 (EN), U2.8 (PS), U2.9 (GND); no longer C1.2, R8.1
- net VBAT_SENSE: no longer R11.2, R12.1
- net at R10.2: now also R8.1, U2.10 (FB)
- net +12V_RAW renamed VBAT_SWITCH
- net +BATT_RAW renamed VBAT
- net 5V_LDO: no longer names the net of C5.1
- net 5V_LDO: now also U2.1 (VAUX)
- net DS18_TEMP renamed BOARD_TEMP
- new net: R18.1, R19.2, U2.7 (UVLO)
- new net: L2.2, U2.3 (L)
- new net VCC: C1.2, JP3.1 (A), L2.1, R11.1, R14.1, R_Shunt1.1
- new net VCC_SENSE: R11.2, R12.1
- no-connect marks 62 -> 48
Other:
- note added: "1S Li-Ion"
- note added: "5V Boost Coverter"
- note added: "Reverse battery protection on boost add fuses?, more ESD protection"
- note added: "TPS61200DRCR"
- note added: "Teensy ADC reads 0-3.3V"
- note added: "VIN: 2.5-4.2V Output: 600mA"
- note added: "Voltage Range Single: 3V-4.2V"
- note removed: "12V VIN MAX 0.08A MAX"
- note removed: "1A IOUT MAX 15V VIN MAX 5V VOUT"
- note removed: "2.54mm 2P Connector"
- note removed: "2S LiPo (7.4V)"
- note removed: "5V Voltage Regulator"
- note removed: "5V Voltage Regulator (Alt.)"
- note removed: "6-32V VIN 3.5A OUT MAX"
- note removed: "AP63357"
- note removed: "ATMEGA328 ADC reads 0-3.3V"
- note removed: "AZ1117IH-5.0TRG1"
- note removed: "Cooling Fan"
- note removed: "Power Option"
- note removed: "UVLO Hi: 5.6V UVLO Lo: 5.18V"
- note removed: "Voltage Range Single: 3V-4.2V Double: 6V-8.4V"
- moved on the sheet: C6, C7, C8, FB1, FB2, FB3, FB4, FB5, FB6, J8
