File: payload/boards/VULCAN/VULCAN.kicad_pcb (KiCad board)
At the start: 2 copper layers, 63.5 x 101.6 mm, 72 parts, among them IC1 LT1001CS8#PBF, J1 XT60PW-M, J2 POWER, J3 I2C, J4 Serial, J5 SPI, J6 GPIO, J7 Screw_Terminal_01x06, J8 Screw_Terminal_01x06, U1 DS18B20+, U2 AZ1117IH-5.0TRG1, U3 MPXV7002DP, U4 AP63357QZV-7, U5 Teensy 4.1, U6 MAX31850KATB+T, U7 MAX31850KATB+T, U8 MAX31850KATB+T

Commit message: updates
Parts:
- removed the R11 at (162.2, 101.2)
- added R12: R, Resistor_SMD:R_0805_2012Metric_Pad1.20x1.40mm_HandSolder, B.Cu at (160.8, 100.1)
- added R2: 62, Resistor_SMD:R_0805_2012Metric_Pad1.20x1.40mm_HandSolder, B.Cu at (183.3, 108.2)
- D4: value BAT165A -> BAT165AX
- turned D2 to 180 degrees
- renumbered D2 to D1, D1 to D2, R9 to R10, R10 to R11, R12 to R13, R13 to R14, R14 to R15, R2 to R3, R3 to R4, R4 to R5, R5 to R6, R6 to R7, R7 to R8, R8 to R9
Connections:
- D2 pad A: /LED_GRN -> Net-(D2-PadA)
- J7 pad 5: /LED_GRN -> Net-(J7-Pin_5)
- U5 pad 15: unconnected-(U5-A1-Pad15) -> /LED_GRN
- U5 pad 23: Net-(U5-A9) -> /LED_EXT
Routing:
- net Net-(D2-PadA): track 0.00 -> 32.9 mm, vias 0 -> 3
- net /LED_GRN: track 26.0 -> 2.31 mm
- net Net-(J7-Pin_5): track 0.00 -> 6.16 mm
- net /LED_EXT: track 0.00 -> 4.76 mm
- net /TC_DATA: track 57.2 -> 60.9 mm
- net Net-(U5-A9): track 1.91 -> 0.00 mm
- net GND: vias 150 -> 157
