File: payload/boards/ARGUS/ARGUS.kicad_sch (KiCad schematic)
At the start: 2 parts, among them J1 XT60PW-M, U1 NRF24L01_Breakout

Commit message: updates
Parts:
- added U2: RASPBERRY_PI_4B_4GB, Module:MODULE_RASPBERRY_PI_4B_4GB, symbol MCU_Module:RASPBERRY_PI_4B_4GB
